File: Converter/Converter.kicad_pcb (KiCad board)
At the start: 2 copper layers, 75 x 75 mm, 6 parts, among them J1 Conn_01x22_Male, J2 Conn_01x22_Male

Commit message: ...
Parts:
- added J3: Conn_01x01_Female, Connector_PinHeader_2.54mm:PinHeader_1x01_P2.54mm_Vertical, F.Cu at (142.9, 90.3)
- J1: footprint Connector_PinHeader_1.00mm:PinHeader_1x22_P1.00mm_Vertical -> Connector_PinHeader_1.27mm:PinHeader_1x23_P1.27mm_Vertical
- moved REF** 15.6 mm to (143.4, 80.4)
- moved REF** 11.6 mm to (145.0, 119.1)
- moved J1 4.52 mm to (111.1, 83.1)
Connections:
- REF** pad 1: (no net) -> GND (x4)
- REF** pad 2: (no net) -> GND (x2)
- REF** pad 3: (no net) -> GND (x2)
Routing:
- net GND: track 0.00 -> 49.1 mm, vias 0 -> 24
- net (no net): track 49.1 -> 0.00 mm, vias 24 -> 0
- net Net-(J1-Pad13): track 20.4 -> 22.9 mm
- net Net-(J1-Pad12): track 19.7 -> 21.9 mm
- net Net-(J1-Pad17): track 22.9 -> 25.0 mm
- net Net-(J1-Pad14): track 21.0 -> 22.9 mm
- net Net-(J1-Pad15): track 21.6 -> 23.4 mm
- net Net-(J1-Pad20): track 24.8 -> 26.5 mm
- net Net-(J1-Pad16): track 22.3 -> 24.0 mm
- net Net-(J1-Pad22): track 26.1 -> 27.6 mm
- net Net-(J1-Pad18): track 23.5 -> 25.0 mm
- net Net-(J1-Pad19): track 24.2 -> 25.6 mm
- net Net-(J1-Pad21): track 25.5 -> 26.6 mm
- net Net-(J1-Pad11): track 20.3 -> 21.3 mm
- net Net-(J1-Pad10): track 21.0 -> 21.9 mm
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- added copper zone on B.Cu, net GND
- added copper zone on F.Cu, net GND
- removed copper zone on B.Cu, net (none)
- removed copper zone on F.Cu, net (none)
Other:
- board size 75 x 75 mm -> 48.3 x 67.1 mm
